Commit message: update for 4 wheel control version

File: example_control_file/2_wheel/ros2_control.xacro (robot description, xacro)
@@ -4,10 +4,10 @@
       <hardware>
         <plugin>epmc_hardware_interface/EPMC_HardwareInterface</plugin>
-        <param name="serial_port">/dev/ttyACM0</param>
+        <param name="serial_port">/dev/ttyUSB0</param>
         <param name="serial_baud_rate">115200</param>
         <param name="serial_timeout_ms">18</param>
         <param name="motor0_wheel_name">left_wheel_joint</param>
         <param name="motor1_wheel_name">right_wheel_joint</param>
-        <param name="cmd_vel_timeout_ms">5000</param>
+        <param name="cmd_vel_timeout_ms">2000</param>
       </hardware>
       <joint name="left_wheel_joint">

File: example_control_file/4_wheel/ros2_control.xacro (robot description, xacro)
@@ -1,14 +1,15 @@
 <?xml version="1.0"?>
 <robot xmlns:xacro="http://www.ros.org/wiki/xacro">
-    <xacro:macro name="epmc_hardware_interface" params="name">
-    <ros2_control name="${name}_front" type="system">
+    <ros2_control name="epmc_hardware_interface" type="system">
       <hardware>
         <plugin>epmc_hardware_interface/EPMC_HardwareInterface</plugin>
-        <param name="serial_port">/dev/ttyACM0</param>
+        <param name="serial_port">/dev/ttyUSB0</param>
         <param name="serial_baud_rate">115200</param>
         <param name="serial_timeout_ms">18</param>
         <param name="motor0_wheel_name">front_left_wheel_joint</param>
         <param name="motor1_wheel_name">front_right_wheel_joint</param>
-        <param name="cmd_vel_timeout_ms">5000</param>
+        <param name="motor2_wheel_name">rear_left_wheel_joint</param>
+        <param name="motor3_wheel_name">rear_right_wheel_joint</param>
+        <param name="cmd_vel_timeout_ms">2000</param>
       </hardware>
       <joint name="front_left_wheel_joint">
@@ -28,15 +29,4 @@
         <state_interface name="velocity"/>
       </joint>
-    </ros2_control>
-    <ros2_control name="${name}_rear" type="system">
-      <hardware>
-        <plugin>epmc_hardware_interface/EPMC_HardwareInterface</plugin>
-        <param name="serial_port">/dev/ttyACM1</param>
-        <param name="serial_baud_rate">115200</param>
-        <param name="serial_timeout_ms">18</param>
-        <param name="motor0_wheel_name">rear_left_wheel_joint</param>
-        <param name="motor1_wheel_name">rear_right_wheel_joint</param>
-        <param name="cmd_vel_timeout_ms">5000</param>
-      </hardware>
       <joint name="rear_left_wheel_joint">
         <command_interface name="velocity">
@@ -56,5 +46,3 @@
       </joint>
     </ros2_control>
-  </xacro:macro>
-  <xacro:epmc_hardware_interface name="epmc_hardware_interface"/>
 </robot>
